File: kicad/soup-soup-soup-sahur.kicad_sch (KiCad schematic)
At the start: 0 parts

Commit message: HOLY PROCRASTINATION :SK: 6 hrs for ts btw
Parts:
- added C1: 220, Capacitor_SMD:C_0805_2012Metric_Pad1.18x1.45mm_HandSolder, symbol Device:C
- added D1: BLUE, LED_SMD:LED_0603_1608Metric_Pad1.05x0.95mm_HandSolder, symbol Device:LED
- added J1: USB_C_Receptacle_PowerOnly_24P, easyeda2kicad:USB-C-SMD_USB-TYPE-C-006, symbol Connector:USB_C_Receptacle_PowerOnly_24P
- added L1: L, 3S:25X48MM_NFC_ANTENNA, symbol Device:L
- added R1: 47, Resistor_SMD:R_0603_1608Metric_Pad0.98x0.95mm_HandSolder, symbol Device:R
- added R2, R3: 5k1, Resistor_SMD:R_0603_1608Metric_Pad0.98x0.95mm_HandSolder, symbol Device:R
- added R4: 18, easyeda2kicad:RES-TH_BD2.2-L6.5-P10.50-D0.6, symbol Device:R
- added SW1: SW_Push, Button_Switch_THT:SW_PUSH_6mm, symbol Switch:SW_Push
- added U1: NT3H2111W0FHKH, 3S:XQFN-8_L1.6-W1.6-P0.50-BL_NT3H2111W0FHKH, symbol 3S:NT3H2111W0FHKH
Connections:
- new net: J1.A5 (CC1), R2.1
- new net: J1.B5 (CC2), R3.1
- new net: R4.1, SW1.2
- new net: C1.1, D1.1 (K), U1.2 (VSS)
- new net: C1.2, R1.1, U1.6 (VCC), U1.7 (VOUT)
- new net: D1.2 (A), R1.2
- new net: L1.1, U1.1 (LA)
- new net: L1.2, U1.8 (LB)
- new net GND: J1.A1 (GND), J1.A12 (GND), J1.B1 (GND), J1.B12 (GND), J1.SH (SHIELD), R2.2, R3.2, R4.2
- new net VBUS: J1.A4 (VBUS), J1.A9 (VBUS), J1.B4 (VBUS), J1.B9 (VBUS), SW1.1
- no-connect marks 0 -> 3
